File: soup-board/pcb/soup_board_kicad/soup_board/soup_board.kicad_sch (KiCad schematic)
At the start: 84 parts

Commit message: finished schematic for v0
Parts:
- removed D39, D40, D41, D42: 1N4148W, Diode_SMD:D_SOD-123, symbol Diode:1N4148W
- removed MX27, MX30, MX33, MX36, MX39, MX42: MX_SW_HS, PCM_marbastlib-mx:SW_MX_HS_1u, symbol PCM_marbastlib-mx:MX_SW_HS
- added I2C_HEADER: ~, symbol soup_parts:I2C_HEADER
- added J1: AudioPlug4, symbol Connector_Audio:AudioPlug4
- added PRO_MICRO1: ~, symbol soup_parts:rp2040_pro_micro
- added R1_PULLUP_10k, R_PULLUP_10K_0: R, symbol Device:R
- added SW2, SW3: RotaryEncoder_Switch, symbol Device:RotaryEncoder_Switch
- added U1: ~, symbol soup_parts:12_PIN_FFC_BREAKOUT
Connections:
- net COL_0: now also PRO_MICRO1.12 (9)
- net COL_1: now also PRO_MICRO1.17 (A3)
- net COL_2: now also PRO_MICRO1.18 (A2)
- net COL_3: now also PRO_MICRO1.19 (A1)
- net COL_4: now also PRO_MICRO1.20 (A0), SW2.S2
- net COL_5: now also PRO_MICRO1.21 (SCK), SW3.S2
- net ROW_0: now also PRO_MICRO1.5 (2)
- net ROW_1: now also PRO_MICRO1.6 (3)
- net ROW_2: now also D13.1 (K), D14.1 (K), D15.1 (K), D16.1 (K), D17.1 (K), D18.1 (K), PRO_MICRO1.7 (4)
- net ROW_3: now also PRO_MICRO1.8 (5)
- net ROW_4: now also PRO_MICRO1.9 (6)
- net ROW_5: now also PRO_MICRO1.10 (7)
- net ROW_6: now also PRO_MICRO1.11 (8)
- net ENC_SWITCH_B_0: now reaches D37.2 (A)
- net ENC_SWITCH_B_0: now also SW3.S1
- net ENC_SWITCH_B_1: now reaches D38.2 (A)
- net ENC_SWITCH_B_1: now also SW2.S1
- new net 3.3V: PRO_MICRO1.16 (VCC), R1_PULLUP_10k.1, R_PULLUP_10K_0.1, U1.12
- new net ENC_ROTARY_A_0: PRO_MICRO1.1 (TX0), SW3.B
- new net ENC_ROTARY_A_1: PRO_MICRO1.22 (CI), SW2.B
- new net ENC_ROTARY_B_0: PRO_MICRO1.2 (RX0), SW3.A
- new net ENC_ROTARY_B_1: PRO_MICRO1.23 (CO), SW2.A
- new net GND: I2C_HEADER.1, J1.T, PRO_MICRO1.14 (GND), SW2.C, SW3.C, U1.11
- new net SCL: I2C_HEADER.4, J1.R2, R1_PULLUP_10k.2, U1.9
- new net SDA: I2C_HEADER.3, J1.R1, R_PULLUP_10K_0.2, U1.10
- new net VCC: J1.S, PRO_MICRO1.13 (RAW)
Other:
- title: (none) -> Soup Board
